File: CC_Load_KiCAD/CC_Load.kicad_sch (KiCad schematic)
At the start: 57 parts, among them J1 VoltSense_Conn, J2 PowerInput_Conn, J3 LED_Conn, J4 Load_Conn, J5 16x2_LCD_Conn, J6 RotEnc_Conn, J7 Fan_Conn, Q1 IRLZ44N, Q2 IRLZ44N, Q3 IRLZ44N, Q4 IRLZ44N, Q5 IRLZ44N, U1 LM7805_TO220, U2 LM358

Commit message: Update schematic and code
Parts:
- removed A2: ~, MyFootprintLibrary:ADC_DAC_Board, symbol MySymbolLibrary:ADC_DAC_Board
- removed C5: 100nF, Capacitor_SMD:C_1206_3216Metric, symbol Device:C
- added C11, C12, C8, C9: 100n, Capacitor_SMD:C_1206_3216Metric, symbol Device:C
- added R19: 22k, Resistor_SMD:R_1206_3216Metric, symbol Device:R
- added R20: 10k, Resistor_SMD:R_1206_3216Metric, symbol Device:R
- added R24: 1k, Resistor_SMD:R_1206_3216Metric, symbol Device:R
- added R25, R26: 100k, Resistor_SMD:R_1206_3216Metric, symbol Device:R
- J1: footprint Connector_PinHeader_2.54mm:PinHeader_1x01_P2.54mm_Vertical -> MyFootprintLibrary:ScrewTerminal_01x02_P5mm
- J2, J4: footprint Connector_PinHeader_2.54mm:PinHeader_1x02_P2.54mm_Vertical -> MyFootprintLibrary:ScrewTerminal_01x02_P5mm
- R22: renamed from R20; value 100R -> 1k
- renumbered C9 to C1, C8 to C10, C1 to C2, C2 to C3, C3 to C4, C4 to C5, R4 to R2, R19 to R21, R21 to R23, R22 to R27, R23 to R28, R24 to R29, R2 to R3, R3 to R4
Connections:
- net +12V: now also J2.2 (Pin_2); no longer J2.1 (Pin_1)
- net GND: now also J2.1 (Pin_1), C11.2, C12.2, C8.2, C9.2, R24.2; no longer J2.2 (Pin_2), J6.5 (Pin_5)
- net curr_sense: now also A1.19 (A0)
- net curr_set: now also C12.1, R26.2
- net temp_sense: now also A1.21 (A2)
- net volt_sense: now also A1.20 (A1)
- net at R22.2, U2.1: now also R19.1; no longer U2.2 (-)
- net at U2.3 (+): now also C8.1, R20.1; no longer R21.1
- net at J6.4 (Pin_4), R28.1: no longer A1.14 (MOSI)
- net at A1.15 (MISO): now also J6.5 (Pin_5)
- new net: R19.2, R24.1, U2.2 (-)
- new net: C9.1, R20.2, R21.1
- new net: C11.1, R25.2, R26.1
- new net: A1.14 (MOSI), R25.1
Other:
- note added: "Bypass cap for op-amp place as close as possible"
- note added: "Low-pass filter"
- note added: "Low-pass filter (PWM to analog voltage)"
- note added: "Non-inverting amplifier (23x gain)"
- moved on the sheet: A1, C10, D1, D2, J1, J2, R1, R18, R2, R21, R22, R3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
